File: DrawBridge.kicad_pcb (KiCad board)
At the start: 2 copper layers, 49.9 x 66.4 mm, 21 parts, among them J1 USB_B, J2 Conn_02x17_Odd_Even, J3 5V DC, J4 FDD POWER, J5 * 12V DC, U1 FT232RL, U2 Arduino Pro Mini, U3 * 7805

Commit message: Increase holes for power cable relief
rev 3b
Other:
- board text added: "PCB for DrawBridge PLUS! by Robert Smith http://amiga.robsmithdev.co.uk Pro Mini rev. 3b design, Damian Woroch"
- board text removed: "PCB for DrawBridge PLUS! by Robert Smith http://amiga.robsmithdev.co.uk Pro Mini rev. 3 design, Damian Woroch, 2022"
Changed lines of the file:
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@@
     (fp_line (start 1.27 -1.27) (end 1.27 8.89) (layer "F.Fab") (width 0.1))
     (fp_line (start -0.635 -1.27) (end 1.27 -1.27) (layer "F.Fab") (width 0.1))
-    (pad "1" thru_hole rect locked (at 0 0 180) (size 1.7 1.7) (drill 1) (layers *.Cu *.Mask)
+    (pad "1" thru_hole rect (at 0 0 180) (size 1.9 1.9) (drill 1.2) (layers *.Cu *.Mask)
       (net 12 "+12V"))
-    (pad "2" thru_hole oval locked (at 0 2.54 180) (size 1.7 1.7) (drill 1) (layers *.Cu *.Mask)
-      (net 1 "GND"))
-    (pad "3" thru_hole oval locked (at 0 5.08 180) (size 1.7 1.7) (drill 1) (layers *.Cu *.Mask)
-      (net 1 "GND"))
-    (pad "4" thru_hole oval locked (at 0 7.62 180) (size 1.7 1.7) (drill 1) (layers *.Cu *.Mask)
+    (pad "2" thru_hole oval (at 0 2.54 180) (size 1.9 1.9) (drill 1.2) (layers *.Cu *.Mask)
+      (net 1 "GND"))
+    (pad "3" thru_hole oval (at 0 5.08 180) (size 1.9 1.9) (drill 1.2) (layers *.Cu *.Mask)
+      (net 1 "GND"))
+    (pad "4" thru_hole oval (at 0 7.62 180) (size 1.9 1.9) (drill 1.2) (layers *.Cu *.Mask)
       (net 6 "+5V"))
     (model "${KISYS3DMOD}/Connector_PinHeader_2.54mm.3dshapes/PinHeader_1x04_P2.54mm_Vertical.wrl"
@@
       (effects (font (size 1 1) (thickness 0.15)))
     )
-    (pad "" np_thru_hole oval (at 0 0 90) (size 7.2 2) (drill oval 7.2 2) (layers F&B.Cu *.Mask))
+    (pad "" np_thru_hole oval (at 0 0 90) (size 7.25 2.1) (drill oval 7.25 2.1) (layers F&B.Cu *.Mask))
   )
   (footprint "Connector_IDC:IDC-Header_2x17_P2.54mm_Vertical" (layer "F.Cu")
@@
     (effects (font (size 0.8 0.8) (thickness 0.1)))
   )
-  (gr_text "PCB for DrawBridge PLUS! by Robert Smith\nhttp://amiga.robsmithdev.co.uk\nPro Mini rev. 3 design, Damian Woroch, 2022" (at 6.3 62.8) (layer "F.SilkS")
+  (gr_text "PCB for DrawBridge PLUS! by Robert Smith\nhttp://amiga.robsmithdev.co.uk\nPro Mini rev. 3b design, Damian Woroch" (at 6.3 62.8) (layer "F.SilkS")
     (effects (font (size 1.08 1.08) (thickness 0.13)) (justify left))
   )

Commit message: Rev 4
Parts:
- removed JP1: 5V SOURCE, Jumper:SolderJumper-3_P1.3mm_Bridged12_Pad1.0x1.5mm
- removed U3: * 7805, Package_TO_SOT_THT:TO-220-3_Vertical
- J2: value Conn_02x17_Odd_Even -> IDC34
- J5: value * 12V DC -> USB FOR INT. MOUNT; footprint Connector_BarrelJack:BarrelJack_Wuerth_6941xx301002 -> Connector_PinHeader_2.54mm:PinHeader_1x04_P2.54mm_Vertical
- moved J4 52.4 mm to (37.5, 56.5)
- moved REF** 52.4 mm to (34.9, 52.7)
- moved J5 26.4 mm to (36.0, 27.2)
- moved REF** 24.6 mm to (13.2, 3.55)
- moved REF** 17.8 mm to (47.4, 51.0), turned to 90 degrees
- moved C1 0.85 mm to (13.7, 14.6)
- moved C2 0.50 mm to (22.8, 9.00)
Connections:
- J1 pad 2: Net-(J1-Pad2) -> Net-(J1-D-)
- J1 pad 3: Net-(J1-Pad3) -> Net-(J1-D+)
- J2 pad 10: (no net) -> unconnected-(J2-Pin_10-Pad10)
- J2 pad 14: (no net) -> unconnected-(J2-Pin_14-Pad14)
- J2 pad 3: (no net) -> unconnected-(J2-Pin_3-Pad3)
- J2 pad 4: (no net) -> unconnected-(J2-Pin_4-Pad4)
- J2 pad 6: (no net) -> unconnected-(J2-Pin_6-Pad6)
- J3 pad 1: Net-(J3-Pad1) -> +5V
- J4 pad 1: +12V -> unconnected-(J4-Pin_1-Pad1)
- J5 pad 1: +12V -> VCC
- J5 pad 2: GND -> Net-(J1-D-)
- J5 pad 3: (no net) -> Net-(J1-D+)
- U1 pad 10: (no net) -> unconnected-(U1-DCD-Pad10)
- U1 pad 12: (no net) -> unconnected-(U1-CBUS4-Pad12)
- U1 pad 13: (no net) -> unconnected-(U1-CBUS2-Pad13)
- U1 pad 14: (no net) -> unconnected-(U1-CBUS3-Pad14)
- U1 pad 15: Net-(J1-Pad3) -> Net-(J1-D+)
- U1 pad 16: Net-(J1-Pad2) -> Net-(J1-D-)
- U1 pad 19: (no net) -> unconnected-(U1-~{RESET}-Pad19)
- U1 pad 22: (no net) -> unconnected-(U1-CBUS1-Pad22)
- U1 pad 23: (no net) -> unconnected-(U1-CBUS0-Pad23)
- U1 pad 27: (no net) -> unconnected-(U1-OSCI-Pad27)
- U1 pad 28: (no net) -> unconnected-(U1-OSCO-Pad28)
- U1 pad 3: (no net) -> unconnected-(U1-RTS-Pad3)
- U1 pad 6: (no net) -> unconnected-(U1-RI-Pad6)
- U1 pad 9: (no net) -> unconnected-(U1-DCR-Pad9)
- U2 pad 1: (no net) -> unconnected-(U2-TX/D1-Pad1)
- U2 pad 2: (no net) -> unconnected-(U2-RX/D0-Pad2)
- U2 pad 21: (no net) -> unconnected-(U2-VCC-Pad21)
- U2 pad 22: (no net) -> unconnected-(U2-~{RESET}-Pad22)
- U2 pad 24: (no net) -> unconnected-(U2-RAW-Pad24)
- U2 pad 3: (no net) -> unconnected-(U2-~{RESET}-Pad3)
Routing:
- net +12V: track 77.1 -> 0.00 mm
- net +5V: track 50.3 -> 8.63 mm
- net Net-(J1-D+): track 0.00 -> 25.9 mm
- net Net-(J1-D-): track 0.00 -> 24.3 mm
- net Net-(J3-Pad1): track 17.6 -> 0.00 mm
- net 5V_7805: track 13.4 -> 0.00 mm
- net Net-(J1-Pad3): track 13.0 -> 0.00 mm
- net VCC: track 41.7 -> 54.6 mm
- net Net-(J1-Pad2): track 11.8 -> 0.00 mm
- net Net-(J2-Pin_28): track 40.9 -> 40.1 mm
- net Net-(J2-Pin_24): track 37.3 -> 38.0 mm
- net Net-(J2-Pin_34): track 62.1 -> 62.8 mm
Other:
- board text added: "GND +5V"
- board text added: "PCB for DrawBridge PLUS! by Robert Smith http://amiga.robsmithdev.co.uk Pro Mini rev. 4 design, Damian Woroch, 2024"
- board text added: "VCC D- D+ GND"
- board text removed: "*optional components, mount these only if floppy disk drive require both 5V and 12V two options to choose from: 1) 7805, set 5V source: 7805, power 12V DC 2) power from 12V DC and 5V DC sockets"
- board text removed: "+12V GND +5V"
- board text removed: "7805/5V DC"
- board text removed: "PCB for DrawBridge PLUS! by Robert Smith http://amiga.robsmithdev.co.uk Pro Mini rev. 3b design, Damian Woroch"
