File: DrawBridge.kicad_sch (KiCad schematic)
At the start: 14 parts, among them J1 USB_B, J2 IDC34, J3 5V DC, J4 FDD POWER, J5 * 12V DC, U1 FT232RL, U2 Arduino Pro Mini, U3 * 7805

Commit message: Rev 4
Parts:
- removed J5: * 12V DC, Connector_BarrelJack:BarrelJack_Wuerth_6941xx301002, symbol Connector:Barrel_Jack
- removed JP1: 5V SOURCE, Jumper:SolderJumper-3_P1.3mm_Bridged12_Pad1.0x1.5mm, symbol Jumper:SolderJumper_3_Bridged12
- removed U3: * 7805, Package_TO_SOT_THT:TO-220-3_Vertical, symbol Regulator_Linear:L7805
- added J5: USB PINS, Connector_PinHeader_2.54mm:PinHeader_1x04_P2.54mm_Vertical, symbol Connector_Generic:Conn_01x04
Connections:
- net +5V: now also J3.1
- net GND: now also J5.4 (Pin_4)
- net VCC: now also J5.1 (Pin_1)
- net at J1.3 (D+), U1.15 (USBD+): now also J5.3 (Pin_3)
- net at J1.2 (D-), U1.16 (USBD-): now also J5.2 (Pin_2)
- net +12V: no longer names the net of J4.1 (Pin_1)
- no-connect marks 27 -> 28
Other:
- moved on the sheet: C1, C2, J3, J4, U1
